File: hardware/Board/Board.kicad_sch (KiCad schematic)
At the start: 9 parts, among them U1 STM32L021K4Tx

Commit message: MCU Board under KiCad
Parts:
- added C10: 10uF, Capacitor_SMD:C_0805_2012Metric_Pad1.18x1.45mm_HandSolder, symbol Device:C_Small
- added C7, C8: 1uF, Capacitor_SMD:C_0805_2012Metric_Pad1.18x1.45mm_HandSolder, symbol Device:C_Small
- added C9: 100nF, Capacitor_SMD:C_0805_2012Metric_Pad1.18x1.45mm_HandSolder, symbol Device:C_Small
- added D3: Green LED, LED_SMD:LED_0603_1608Metric_Pad1.05x0.95mm_HandSolder, symbol Device:LED_Small
- added J1: Conn_02x07_Odd_Even, Connector_PinHeader_1.27mm:PinHeader_2x07_P1.27mm_Vertical_SMD, symbol Connector_Generic:Conn_02x07_Odd_Even
- added J2: Power, Connector_JST:JST_XH_B2B-XH-A_1x02_P2.50mm_Vertical, symbol Connector_Generic:Conn_01x02
- added J3: Output, Connector_JST:JST_XH_B2B-XH-A_1x02_P2.50mm_Vertical, symbol Connector_Generic:Conn_01x02
- added J4: Input, Connector_JST:JST_XH_B2B-XH-A_1x02_P2.50mm_Vertical, symbol Connector_Generic:Conn_01x02
- added R4: 1K, Resistor_SMD:R_0805_2012Metric_Pad1.20x1.40mm_HandSolder, symbol Device:R_Small
- added U2: MCP4801, Package_SO:SOIC-8_3.9x4.9mm_P1.27mm, symbol Analog_DAC:MCP4801
- added U3: BU33SD5WG-TR, Package_TO_SOT_SMD:SOT-23-5, symbol Regulator_Linear:MCP1802x-xx02xOT
Connections:
- net +3.3V: now also C8.1, D3.2 (A), J1.3 (Pin_3), U3.5 (VOUT)
- net +3.3VA: now also C10.1, C9.1, U2.1 (Vdd), U2.6 (~{SHDN})
- net ADC_IN1: now also U1.8 (PA2), J4.1 (Pin_1)
- net DAC_nCS: now also U1.10 (PA4), U2.2 (~{CS})
- net DAC_nLDAC: now also U2.5 (~{LDAC})
- net GND: now also C10.2, C9.2, J1.11 (Pin_11), J1.5 (Pin_5), J1.7 (Pin_7), J2.2 (Pin_2), J3.2 (Pin_2), J4.2 (Pin_2), R4.2, U2.7 (Vss)
- net LED_STATUS: now also U1.18 (PA8)
- net SPI1_CSK: now also U1.11 (PA5)
- net SPI_MOSI: now also U1.13 (PA7), U2.4 (SDI)
- net SWDIO: now also J1.4 (Pin_4)
- net USART2_RX: now also J1.13 (Pin_13)
- net USART2_TX: now also J1.14 (Pin_14)
- new net: D3.1 (K), R4.1
- new net: C7.2, C8.2, U3.2 (GND)
- new net +5V: C7.1, J2.1 (Pin_1), U3.1 (VIN), U3.3 (~{SHDN})
- new net DAC_OUT: J3.1 (Pin_1), U2.8 (Vout)
- new net NRST: J1.12 (Pin_12)
- new net SPI1_SCK: U2.3 (SCK)
- new net SWDCLK: J1.6 (Pin_6)
- no-connect marks 0 -> 5
Other:
- note added: "DAC MCP4801"
- note added: "IO Connector"
- note added: "Power supply"
- note added: "SWD Connector"

Commit message: Board schematic
Parts:
- added H1, H2, H3, H4: MountingHole_Pad, MountingHole:MountingHole_3.2mm_M3_Pad, symbol Mechanical:MountingHole_Pad
- added R2: 100k, Resistor_SMD:R_0805_2012Metric_Pad1.20x1.40mm_HandSolder, symbol Device:R_Small
- C1: value 4u7 -> 4uF; footprint (none) -> Capacitor_SMD:C_0805_2012Metric_Pad1.18x1.45mm_HandSolder
- C2, C3, C5, C6: footprint (none) -> Capacitor_SMD:C_0805_2012Metric_Pad1.18x1.45mm_HandSolder
- C4: footprint (none) -> Capacitor_SMD:C_0805_2012Metric
- C7: footprint Capacitor_SMD:C_0805_2012Metric_Pad1.18x1.45mm_HandSolder -> Capacitor_SMD:C_0805_2012Metric
- D1: footprint (none) -> LED_SMD:LED_0603_1608Metric_Pad1.05x0.95mm_HandSolder
- L1: footprint (none) -> Inductor_SMD:L_0805_2012Metric_Pad1.05x1.20mm_HandSolder
Connections:
- net NSRT is gone; now on net NRST: C6.1, U1.4 (NRST)
- net SPI1_CSK is gone; now on net SPI1_SCK: U1.11 (PA5)
- net SWDCK is gone; now on net SWDCLK: U1.24 (PA14)
- net GND: now also C7.2, C8.2, U3.2 (GND), H1.1, H2.1, H3.1, H4.1, R2.2
- net at U1.31 (PB9): now also R2.1
- no-connect marks 5 -> 20
